Commit message: Add real robot launch file

File: alicia_d_moveit/config/Alicia_D_v5_5_gripper_100mm.urdf.xacro (robot description, xacro)
@@ -2,9 +2,23 @@
 <robot xmlns:xacro="http://www.ros.org/wiki/xacro" name="Alicia_D_v5_5_gripper_100mm">
     <xacro:arg name="initial_positions_file" default="initial_positions.yaml" />
+    <xacro:arg name="hw_port" default="/dev/ttyCH341USB0" />
+    <xacro:arg name="hw_baud_rate" default="1000000" />
+    <xacro:arg name="hw_debug_mode" default="false" />
+    <xacro:arg name="hw_servo_count" default="9" />
+    <xacro:arg name="hw_gripper_type" default="100mm" />
+    <xacro:arg name="hw_firmware_version" default="auto" />
     <!-- Import alicia_d_descriptions urdf file for v5_5 100mm -->
     <xacro:include filename="$(find alicia_d_descriptions)/urdf/Alicia_D_v5_5/Alicia_D_gripper_100mm.urdf" />
     <!-- Import control_xacro -->
     <xacro:include filename="alicia_d_descriptions.ros2_control.xacro" />
-    <!-- Use FakeSystem for demo mode -->
-    <xacro:alicia_d_descriptions_ros2_control name="FakeSystem" initial_positions_file="$(arg initial_positions_file)"/>
+    <!-- Use ros2_control with configurable hardware interface -->
+    <xacro:alicia_d_descriptions_ros2_control
+        name="AliciaDHardware"
+        initial_positions_file="$(arg initial_positions_file)"
+        hw_port="$(arg hw_port)"
+        hw_baud_rate="$(arg hw_baud_rate)"
+        hw_debug_mode="$(arg hw_debug_mode)"
+        hw_servo_count="$(arg hw_servo_count)"
+        hw_gripper_type="$(arg hw_gripper_type)"
+        hw_firmware_version="$(arg hw_firmware_version)"/>
 </robot>

File: alicia_d_moveit/config/Alicia_D_v5_6_gripper_100mm.urdf.xacro (robot description, xacro)
@@ -2,9 +2,23 @@
 <robot xmlns:xacro="http://www.ros.org/wiki/xacro" name="Alicia_D_v5_6_gripper_100mm">
     <xacro:arg name="initial_positions_file" default="initial_positions.yaml" />
+    <xacro:arg name="hw_port" default="/dev/ttyCH341USB0" />
+    <xacro:arg name="hw_baud_rate" default="1000000" />
+    <xacro:arg name="hw_debug_mode" default="false" />
+    <xacro:arg name="hw_servo_count" default="9" />
+    <xacro:arg name="hw_gripper_type" default="100mm" />
+    <xacro:arg name="hw_firmware_version" default="auto" />
     <!-- Import alicia_d_descriptions urdf file for v5_6 100mm -->
     <xacro:include filename="$(find alicia_d_descriptions)/urdf/Alicia_D_v5_6/Alicia_D_gripper_100mm.urdf" />
     <!-- Import control_xacro -->
     <xacro:include filename="alicia_d_descriptions.ros2_control.xacro" />
-    <!-- Use FakeSystem for demo mode -->
-    <xacro:alicia_d_descriptions_ros2_control name="FakeSystem" initial_positions_file="$(arg initial_positions_file)"/>
+    <!-- Use ros2_control with configurable hardware interface -->
+    <xacro:alicia_d_descriptions_ros2_control
+        name="AliciaDHardware"
+        initial_positions_file="$(arg initial_positions_file)"
+        hw_port="$(arg hw_port)"
+        hw_baud_rate="$(arg hw_baud_rate)"
+        hw_debug_mode="$(arg hw_debug_mode)"
+        hw_servo_count="$(arg hw_servo_count)"
+        hw_gripper_type="$(arg hw_gripper_type)"
+        hw_firmware_version="$(arg hw_firmware_version)"/>
 </robot>

File: alicia_d_moveit/config/Alicia_D_v5_6_gripper_50mm.urdf.xacro (robot description, xacro)
@@ -2,9 +2,23 @@
 <robot xmlns:xacro="http://www.ros.org/wiki/xacro" name="Alicia_D_v5_6_gripper_50mm">
     <xacro:arg name="initial_positions_file" default="initial_positions.yaml" />
+    <xacro:arg name="hw_port" default="/dev/ttyCH341USB0" />
+    <xacro:arg name="hw_baud_rate" default="1000000" />
+    <xacro:arg name="hw_debug_mode" default="false" />
+    <xacro:arg name="hw_servo_count" default="9" />
+    <xacro:arg name="hw_gripper_type" default="50mm" />
+    <xacro:arg name="hw_firmware_version" default="auto" />
     <!-- Import alicia_d_descriptions urdf file for v5_6 50mm -->
     <xacro:include filename="$(find alicia_d_descriptions)/urdf/Alicia_D_v5_6/Alicia_D_gripper_50mm.urdf" />
     <!-- Import control_xacro -->
     <xacro:include filename="alicia_d_descriptions.ros2_control.xacro" />
-    <!-- Use FakeSystem for demo mode -->
-    <xacro:alicia_d_descriptions_ros2_control name="FakeSystem" initial_positions_file="$(arg initial_positions_file)"/>
+    <!-- Use ros2_control with configurable hardware interface -->
+    <xacro:alicia_d_descriptions_ros2_control
+        name="AliciaDHardware"
+        initial_positions_file="$(arg initial_positions_file)"
+        hw_port="$(arg hw_port)"
+        hw_baud_rate="$(arg hw_baud_rate)"
+        hw_debug_mode="$(arg hw_debug_mode)"
+        hw_servo_count="$(arg hw_servo_count)"
+        hw_gripper_type="$(arg hw_gripper_type)"
+        hw_firmware_version="$(arg hw_firmware_version)"/>
 </robot>

File: alicia_d_moveit/config/alicia_d_descriptions.ros2_control.xacro (robot description, xacro)
@@ -1,9 +1,18 @@
 <?xml version="1.0"?>
 <robot xmlns:xacro="http://www.ros.org/wiki/xacro">
-    <xacro:macro name="alicia_d_descriptions_ros2_control" params="name initial_positions_file">
+    <xacro:macro name="alicia_d_descriptions_ros2_control" params="name initial_positions_file
+                 hw_port:=/dev/ttyCH341USB0 hw_baud_rate:=1000000
+                 hw_debug_mode:=false hw_servo_count:=9
+                 hw_gripper_type:=50mm hw_firmware_version:=auto">
         <xacro:property name="initial_positions" value="${xacro.load_yaml(initial_positions_file)['initial_positions']}"/>
         <ros2_control name="${name}" type="system">
             <hardware>
-                <plugin>mock_components/GenericSystem</plugin>
+                <plugin>alicia_d_driver/AliciaDHardwareInterface</plugin>
+                <param name="port">${hw_port}</param>
+                <param name="baud_rate">${hw_baud_rate}</param>
+                <param name="debug_mode">${hw_debug_mode}</param>
+                <param name="servo_count">${hw_servo_count}</param>
+                <param name="gripper_type">${hw_gripper_type}</param>
+                <param name="firmware_version">${hw_firmware_version}</param>
             </hardware>
             <joint name="Joint1">
