Commit message: Update the moveit configurations

File: alicia_d_descriptions/urdf/Alicia_D_v5_6/Alicia_D_v5_6_gripper_100mm.urdf (robot description, URDF)
Before this commit: robot Alicia_D_v5_6_gripper_100mm, 10 links, 9 joints
Joints:
- joint left_finger: mimic (none) -> joint=Gripper multiplier=-1 offset=0

File: alicia_d_moveit/config/Alicia_D_v5_6_gripper_100mm.urdf.xacro (robot description, xacro)
@@ -2,13 +2,10 @@
 <robot xmlns:xacro="http://www.ros.org/wiki/xacro" name="Alicia_D_v5_6_gripper_100mm">
     <xacro:arg name="initial_positions_file" default="initial_positions.yaml" />
-    <xacro:arg name="hw_port" default="/dev/ttyUSB0" />
-    <xacro:arg name="hw_baud_rate" default="1000000" />
+    <xacro:arg name="hw_port" default="" />
     <xacro:arg name="hw_debug_mode" default="false" />
-    <xacro:arg name="hw_servo_count" default="9" />
     <xacro:arg name="hw_gripper_type" default="100mm" />
-    <xacro:arg name="hw_firmware_version" default="auto" />
     <xacro:arg name="hw_default_speed_rad_s" default="0.349" />
     <!-- Import alicia_d_descriptions urdf file for v5_6 100mm -->
-    <xacro:include filename="$(find alicia_d_descriptions)/urdf/Alicia_D_v5_6/Alicia_D_gripper_100mm.urdf" />
+    <xacro:include filename="$(find alicia_d_descriptions)/urdf/Alicia_D_v5_6/Alicia_D_v5_6_gripper_100mm.urdf" />
     <!-- Import control_xacro -->
     <xacro:include filename="alicia_d_descriptions.ros2_control.xacro" />
@@ -18,9 +15,5 @@
         initial_positions_file="$(arg initial_positions_file)"
         hw_port="$(arg hw_port)"
-        hw_baud_rate="$(arg hw_baud_rate)"
-        hw_debug_mode="$(arg hw_debug_mode)"
-        hw_servo_count="$(arg hw_servo_count)"
         hw_gripper_type="$(arg hw_gripper_type)"
-        hw_firmware_version="$(arg hw_firmware_version)"
         hw_default_speed_rad_s="$(arg hw_default_speed_rad_s)"/>
 </robot>

File: alicia_d_moveit/config/Alicia_D_v5_6_gripper_50mm.urdf.xacro (robot description, xacro)
@@ -2,13 +2,9 @@
 <robot xmlns:xacro="http://www.ros.org/wiki/xacro" name="Alicia_D_v5_6_gripper_50mm">
     <xacro:arg name="initial_positions_file" default="initial_positions.yaml" />
-    <xacro:arg name="hw_port" default="/dev/ttyUSB0" />
-    <xacro:arg name="hw_baud_rate" default="1000000" />
-    <xacro:arg name="hw_debug_mode" default="false" />
-    <xacro:arg name="hw_servo_count" default="9" />
+    <xacro:arg name="hw_port" default="" />
     <xacro:arg name="hw_gripper_type" default="50mm" />
-    <xacro:arg name="hw_firmware_version" default="auto" />
     <xacro:arg name="hw_default_speed_rad_s" default="0.349" />
     <!-- Import alicia_d_descriptions urdf file for v5_6 50mm -->
-    <xacro:include filename="$(find alicia_d_descriptions)/urdf/Alicia_D_v5_6/Alicia_D_gripper_50mm.urdf" />
+    <xacro:include filename="$(find alicia_d_descriptions)/urdf/Alicia_D_v5_6/Alicia_D_v5_6_gripper_50mm.urdf" />
     <!-- Import control_xacro -->
     <xacro:include filename="alicia_d_descriptions.ros2_control.xacro" />
@@ -18,9 +14,5 @@
         initial_positions_file="$(arg initial_positions_file)"
         hw_port="$(arg hw_port)"
-        hw_baud_rate="$(arg hw_baud_rate)"
-        hw_debug_mode="$(arg hw_debug_mode)"
-        hw_servo_count="$(arg hw_servo_count)"
         hw_gripper_type="$(arg hw_gripper_type)"
-        hw_firmware_version="$(arg hw_firmware_version)"
         hw_default_speed_rad_s="$(arg hw_default_speed_rad_s)"/>
 </robot>

File: alicia_d_moveit/config/alicia_d_descriptions.ros2_control.fake.xacro (robot description, xacro)
@@ -1,16 +1,10 @@
 <?xml version="1.0"?>
 <robot xmlns:xacro="http://www.ros.org/wiki/xacro">
-    <xacro:macro name="alicia_d_descriptions_ros2_control" params="name initial_positions_file
-                 hw_port:=
-                 hw_debug_mode:=false
-                 hw_gripper_type:=50mm
-                 hw_default_speed_rad_s:=0.349">
+    <xacro:macro name="alicia_d_descriptions_ros2_control" params="name initial_positions_file">
         <xacro:property name="initial_positions" value="${xacro.load_yaml(initial_positions_file)['initial_positions']}"/>
         <ros2_control name="${name}" type="system">
             <hardware>
-                <plugin>alicia_d_driver/AliciaDHardwareInterface</plugin>
-                <param name="port">${hw_port}</param>
-                <param name="gripper_type">${hw_gripper_type}</param>
-                <param name="default_speed_rad_s">${hw_default_speed_rad_s}</param>
+                <plugin>fake_components/GenericSystem</plugin>
+                <param name="state_following_offset">0.0</param>
             </hardware>
             <joint name="Joint1">

File: alicia_d_moveit/config/alicia_d_descriptions.urdf.xacro (robot description, xacro)
@@ -3,5 +3,5 @@
     <xacro:arg name="initial_positions_file" default="initial_positions.yaml" />
     <!-- Import alicia_d_descriptions urdf file -->
-    <xacro:include filename="$(find alicia_d_descriptions)/urdf/Alicia_D_v5_6/Alicia_D_gripper_50mm.urdf" />
+    <xacro:include filename="$(find alicia_d_descriptions)/urdf/Alicia_D_v5_6/Alicia_D_v5_6_gripper_50mm.urdf" />
     <!-- Import control_xacro -->
     <xacro:include filename="alicia_d_descriptions.ros2_control.xacro" />

Commit message: Upload real robot control

File: alicia_d_descriptions/urdf/Alicia_D_v5_6/Alicia_D_v5_6_gripper_100mm.urdf (robot description, URDF)
Before this commit: robot Alicia_D_v5_6_gripper_100mm, 10 links, 9 joints
Joints:
- joint Joint1: axis -0.0397713509246861 0 -0.999208806829496 -> -0.0397713509246861 0 0.999208806829496; limit lower=-2.7925 upper=2.7525 effort=5 velocity=12 -> lower=-2.749 upper=2.749 effort=5 velocity=12
- joint Joint2: axis 0 0 1 -> 0 0 -1; limit lower=-2 upper=2 effort=5 velocity=12 -> lower=-1.57 upper=1.57 effort=5 velocity=12
- joint Joint3: axis 0 0 1 -> 0 0 -1; limit lower=-2.8 upper=0.38 effort=5 velocity=12 -> lower=-0.78 upper=3.14159 effort=5 velocity=12
- joint Joint5: limit lower=-1.5 upper=1.5 effort=5 velocity=12 -> lower=-1.57 upper=1.57 effort=5 velocity=12

File: alicia_d_descriptions/urdf/Alicia_D_v5_6/Alicia_D_v5_6_gripper_50mm.urdf (robot description, URDF)
Before this commit: robot Alicia_D_v5_6_gripper_50mm, 10 links, 9 joints
Joints:
- joint Joint1: axis -0.0397713509246861 0 -0.999208806829496 -> -0.0397713509246861 0 0.999208806829496; limit lower=-2.7925 upper=2.7525 effort=5 velocity=12 -> lower=-2.749 upper=2.749 effort=5 velocity=12
- joint Joint2: axis 0 0 1 -> 0 0 -1; limit lower=-2 upper=2 effort=5 velocity=12 -> lower=-1.57 upper=1.57 effort=5 velocity=12
- joint Joint3: axis 0 0 1 -> 0 0 -1; limit lower=-2.8 upper=0.38 effort=5 velocity=12 -> lower=-0.78 upper=3.14159 effort=5 velocity=12
- joint Joint5: limit lower=-1.5 upper=1.5 effort=5 velocity=12 -> lower=-1.57 upper=1.57 effort=5 velocity=12

Commit message: Update the documentation and speed unit

File: alicia_d_descriptions/urdf/Alicia_D_v5_6/Alicia_D_v5_6_gripper_100mm.urdf (robot description, URDF)
Before this commit: robot Alicia_D_v5_6_gripper_100mm, 10 links, 9 joints
Joints:
- removed joint left_finger
- added joint right_finger: type prismatic, parent Link6, child right_gripper, origin xyz=-0.0002 0.050502 0.13098 rpy=-1.5708 0 0, axis 0 0 1, limit lower=-0.05 upper=0 effort=5 velocity=12, mimic joint=Gripper multiplier=-1 offset=0
- joint Gripper: axis 0 0 1 -> 0 0 -1; child right_gripper -> left_gripper; limit lower=-0.05 upper=0 effort=5 velocity=12 -> lower=0 upper=0.05 effort=5 velocity=12; origin xyz=-0.0002 0.050502 0.13098 rpy=-1.5708 0 0 -> xyz=-0.000200000000001033 -0.050497849845622 0.130979659620446 rpy=1.5707963267949 0 0

File: alicia_d_descriptions/urdf/Alicia_D_v5_6/Alicia_D_v5_6_gripper_50mm.urdf (robot description, URDF)
Before this commit: robot Alicia_D_v5_6_gripper_50mm, 10 links, 9 joints
Joints:
- removed joint left_finger
- added joint right_finger: type prismatic, parent Link6, child right_gripper, origin xyz=0.0002 0.0255 0.13098 rpy=-1.5708 0 0, axis 0 0 1, limit lower=-0.025 upper=0 effort=5 velocity=12, mimic joint=Gripper multiplier=-1 offset=0
- joint Gripper: axis 0 0 1 -> 0 0 -1; child right_gripper -> left_gripper; limit lower=-0.025 upper=0 effort=5 velocity=12 -> lower=0 upper=0.025 effort=5 velocity=12; origin xyz=0.0002 0.0255 0.13098 rpy=-1.5708 0 0 -> xyz=0.0002 -0.0255 0.13098 rpy=1.5708 0 0

File: alicia_d_moveit/config/Alicia_D_v5_6_gripper_100mm.urdf.xacro (robot description, xacro)
@@ -5,5 +5,5 @@
     <xacro:arg name="hw_debug_mode" default="false" />
     <xacro:arg name="hw_gripper_type" default="100mm" />
-    <xacro:arg name="hw_default_speed_rad_s" default="0.349" />
+    <xacro:arg name="hw_default_speed_deg_s" default="20.0" />
     <!-- Import alicia_d_descriptions urdf file for v5_6 100mm -->
     <xacro:include filename="$(find alicia_d_descriptions)/urdf/Alicia_D_v5_6/Alicia_D_v5_6_gripper_100mm.urdf" />
@@ -16,4 +16,4 @@
         hw_port="$(arg hw_port)"
         hw_gripper_type="$(arg hw_gripper_type)"
-        hw_default_speed_rad_s="$(arg hw_default_speed_rad_s)"/>
+        hw_default_speed_deg_s="$(arg hw_default_speed_deg_s)"/>
 </robot>

File: alicia_d_moveit/config/Alicia_D_v5_6_gripper_50mm.urdf.xacro (robot description, xacro)
@@ -4,5 +4,5 @@
     <xacro:arg name="hw_port" default="" />
     <xacro:arg name="hw_gripper_type" default="50mm" />
-    <xacro:arg name="hw_default_speed_rad_s" default="0.349" />
+    <xacro:arg name="hw_default_speed_deg_s" default="20.0" />
     <!-- Import alicia_d_descriptions urdf file for v5_6 50mm -->
     <xacro:include filename="$(find alicia_d_descriptions)/urdf/Alicia_D_v5_6/Alicia_D_v5_6_gripper_50mm.urdf" />
@@ -15,4 +15,4 @@
         hw_port="$(arg hw_port)"
         hw_gripper_type="$(arg hw_gripper_type)"
-        hw_default_speed_rad_s="$(arg hw_default_speed_rad_s)"/>
+        hw_default_speed_deg_s="$(arg hw_default_speed_deg_s)"/>
 </robot>

File: alicia_d_moveit/config/alicia_d_descriptions.ros2_control.xacro (robot description, xacro)
@@ -5,5 +5,5 @@
                  hw_debug_mode:=false
                  hw_gripper_type:=50mm
-                 hw_default_speed_rad_s:=0.349">
+                 hw_default_speed_deg_s:=20.0">
         <xacro:property name="initial_positions" value="${xacro.load_yaml(initial_positions_file)['initial_positions']}"/>
         <ros2_control name="${name}" type="system">
@@ -12,5 +12,5 @@
                 <param name="port">${hw_port}</param>
                 <param name="gripper_type">${hw_gripper_type}</param>
-                <param name="default_speed_rad_s">${hw_default_speed_rad_s}</param>
+                <param name="default_speed_deg_s">${hw_default_speed_deg_s}</param>
             </hardware>
             <joint name="Joint1">
